File: pcb/RFID_CC_READER/PN532_Shield.brd (EAGLE design)
At the start: 86.2 x 53.4 mm, 44 parts, among them U1 PN532, U2 ADP122(3.3V), U3 STM32F103C8T6, Y1 27.12MHz

Commit message: library updates
Connections:
- new net S$1: C23.2, C27.2, C3.2, C7.2, C9.2
- new net S$2: U3.8
- new net S$3: C10.1, C8.1
- net GND: no longer C10.1, C23.2, C27.2, C3.2, C7.2, C8.1, C9.2, L5.MIDDLE_PIN, U3.8, U4.GND1
- net N$2: no longer L4.2
- net VDD: no longer C21.1
Routing:
- net GND: track 284.2 -> 177.4 mm, vias 4 -> 0
- net S$1: track 0.00 -> 52.4 mm, vias 0 -> 2
- net S$2: track 0.00 -> 29.9 mm, vias 0 -> 2
- net S$3: track 0.00 -> 18.8 mm
- net N$3: track 66.3 -> 52.8 mm
- net VDD: track 123.9 -> 121.9 mm
- net N$2: track 17.1 -> 16.6 mm
