File: pcb/RFID_CC_READER/PN532_Shield.sch (EAGLE design)
At the start: 44 parts, among them U1 PN532, U2 ADP122(3.3V), U3 STM32F103C8T6, Y1 27.12MHz

Commit message: library updates
Parts:
- added R7: 10K, microbuilder:RESISTOR0805
Connections:
- new net N$15: C27.P$2, Q1.1, U3.PC15-OSC32_OUT
- new net N$16: C23.P$1, C27.P$1
- new net N$17: R5.2, U4.D+
- new net N$18: R6.1, U4.D-
- new net N$6: C23.P$2, Q1.2, U3.PC14-OSC32_IN
- new net USB_D_MINUS: R6.2, U3.PA11
- new net USB_D_PLUS: R5.1, R7.1, U3.PA12
- net GND: now also U3.BOOT0, U3.PB2
- net VCC: now also R7.2
Other:
- moved on the sheet: C23, C27, Q1, R5, R6
